File: heater/heater.kicad_pcb (KiCad board)
At the start: 2 copper layers, 100 x 100 mm, 7 parts, among them J1 ED550/4DS

Commit message: Added data matrix codes to PCBs for easy identification
Parts:
- added G***: LOGO, LOGO, B.Cu at (145.0, 109.0)
Changed lines of the file:
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@@
+		)
+	)
+	(footprint "LOGO"
+		(layer "B.Cu")
+		(at 145 109 180)
+		(property "Reference" "G***"
+			(at 0 0 0)
+			(layer "B.SilkS")
+			(hide yes)
+			(effects
+				(font
+					(size 1.5 1.5)
+					(thickness 0.3)
+				)
+				(justify mirror)
+			)
+		)
+		(property "Value" "LOGO"
+			(at 0.75 0 0)
+			(layer "B.SilkS")
+			(hide yes)
+			(effects
+				(font
+					(size 1.5 1.5)
+					(thickness 0.3)
+				)
+				(justify mirror)
+			)
+		)
+		(property "Footprint" ""
+			(at 0 0 0)
+			(layer "B.Fab")
+			(hide yes)
+			(effects
+				(font
+					(size 1.27 1.27)
+					(thickness 0.15)
+				)
+				(justify mirror)
+			)
+		)
+		(property "Datasheet" ""
+			(at 0 0 0)
+			(layer "B.Fab")
+			(hide yes)
+			(effects
+				(font
+					(size 1.27 1.27)
+					(thickness 0.15)
+				)
+				(justify mirror)
+			)
+		)
+		(property "Description" ""
+			(at 0 0 0)
+			(layer "B.Fab")
+			(hide yes)
+			(effects
+				(font
+					(size 1.27 1.27)
+					(thickness 0.15)
+				)
+				(justify mirror)
+			)
+		)
+		(attr board_only exclude_from_pos_files exclude_from_bom)
+		(fp_poly
+			(pts
+				(xy 2.883995 -3.248837) (xy 2.883995 -3.61368) (xy 2.536526 -3.61368) (xy 2.189056 -3.61368) (xy 2.189056 -3.248837)
+				(xy 2.189056 -2.883995) (xy 2.536526 -2.883995) (xy 2.883995 -2.883995)
+			)
+			(stroke
+				(width 0)
+				(type solid)
+			)
+			(fill solid)
+			(layer "B.SilkS")
+		)
+		(fp_poly
+			(pts
+				(xy 2.189056 1.094528) (xy 2.189056 0.729685) (xy 1.459371 0.729685) (xy 0.729686 0.729685) (xy 0.729686 1.094528)
+				(xy 0.729686 1.45937) (xy 1.459371 1.45937) (xy 2.189056 1.45937)
+			)
+			(stroke
+				(width 0)
+				(type solid)
+			)
+			(fill solid)
+			(layer "B.SilkS")
+		)
+		(fp_poly
+			(pts
+				(xy -2.883994 -0.364843) (xy -2.883994 -0.729686) (xy -3.248837 -0.729686) (xy -3.61368 -0.729686)
+				(xy -3.61368 -0.364843) (xy -3.61368 0) (xy -3.248837 0) (xy -2.883994 0)
+			)
+			(stroke
+				(width 0)
+				(type solid)
+			)
+			(fill solid)
+			(layer "B.SilkS")
+		)
+		(fp_poly
+			(pts
+				(xy 2.189056 -0.729686) (xy 2.189056 -1.459371) (xy 1.824214 -1.459371) (xy 1.459371 -1.459371)
+				(xy 1.459371 -1.094528) (xy 1.459371 -0.729686) (xy 1.094528 -0.729686) (xy 0.729686 -0.729686)
+				(xy 0.729686 -1.094528) (xy 0.729686 -1.459371) (xy 0.364843 -1.459371) (xy 0 -1.459371) (xy 0 -0.729686)
+				(xy 0 0) (xy 1.094528 0) (xy 2.189056 0)
+			)
+			(stroke
+				(width 0)
+				(type solid)
+			)
+			(fill solid)
+			(layer "B.SilkS")
+		)
+		(fp_poly
+			(pts
+				(xy 1.459371 -2.536526) (xy 1.459371 -2.883995) (xy 1.094528 -2.883995) (xy 0.729686 -2.883995)
+				(xy 0.729686 -3.248837) (xy 0.729686 -3.61368) (xy 0 -3.61368) (xy -0.729685 -3.61368) (xy -0.729685 -3.248837)
+				(xy -0.729685 -2.883995) (xy 0 -2.883995) (xy 0.729686 -2.883995) (xy 0.729686 -2.536526) (xy 0.729686 -2.189056)
+				(xy 1.094528 -2.189056) (xy 1.459371 -2.189056)
+			)
+			(stroke
+				(width 0)
+				(type solid)
+			)
+			(fill solid)
+			(layer "B.SilkS")
+		)
+		(fp_poly
+			(pts
+				(xy -2.189056 -1.459371) (xy -2.189056 -2.189056) (xy -2.536525 -2.189056) (xy -2.883994 -2.189056)
+				(xy -2.883994 -2.536526) (xy -2.883994 -2.883995) (xy -2.536525 -2.883995) (xy -2.189056 -2.883995)
+				(xy -2.189056 -2.536526) (xy -2.189056 -2.189056) (xy -1.824213 -2.189056) (xy -1.45937 -2.189056)
+				(xy -1.45937 -2.901368) (xy -1.45937 -3.61368) (xy -2.536525 -3.61368) (xy -3.61368 -3.61368) (xy -3.61368 -2.901368)
+				(xy -3.61368 -2.189056) (xy -3.248837 -2.189056) (xy -2.883994 -2.189056) (xy -2.883994 -1.459371)
+				(xy -2.883994 -0.729686) (xy -2.536525 -0.729686) (xy -2.189056 -0.729686)
+			)
+			(stroke
+				(width 0)
+				(type solid)
+			)
+			(fill solid)
+			(layer "B.SilkS")
+		)
+		(fp_poly
+			(pts
+				(xy 5.003557 0) (xy 5.003557 -5.003557) (xy 0 -5.003557) (xy -5.003556 -5.003557) (xy -5.003556 0)
+				(xy -4.343365 0) (xy -4.343365 -4.343366) (xy 0 -4.343366) (xy 4.343366 -4.343366) (xy 4.343366 -3.978523)
+				(xy 4.343366 -3.61368) (xy 3.978523 -3.61368) (xy 3.61368 -3.61368) (xy 3.61368 -3.248837) (xy 3.61368 -2.883995)
+				(xy 3.978523 -2.883995) (xy 4.343366 -2.883995) (xy 4.343366 -2.536526) (xy 4.343366 -2.189056)
+				(xy 3.978523 -2.189056) (xy 3.61368 -2.189056) (xy 3.61368 -2.536526) (xy 3.61368 -2.883995) (xy 3.248837 -2.883995)
+				(xy 2.883995 -2.883995) (xy 2.883995 -1.80684) (xy 2.883995 -1.094528) (xy 3.61368 -1.094528) (xy 3.61368 -1.459371)
+				(xy 3.978523 -1.459371) (xy 4.343366 -1.459371) (xy 4.343366 -1.094528) (xy 4.343366 -0.729686)
+				(xy 3.978523 -0.729686) (xy 3.61368 -0.729686) (xy 3.61368 -1.094528) (xy 2.883995 -1.094528) (xy 2.883995 -0.729686)
+				(xy 3.248837 -0.729686) (xy 3.61368 -0.729686) (xy 3.61368 -0.364843) (xy 3.61368 0) (xy 3.978523 0)
+				(xy 4.343366 0) (xy 4.343366 0.364842) (xy 4.343366 0.729685) (xy 3.61368 0.729685) (xy 2.883995 0.729685)
+				(xy 2.883995 1.094528) (xy 2.883995 1.45937) (xy 2.536526 1.45937) (xy 2.189056 1.45937) (xy 2.189056 1.824213)
+				(xy 3.61368 1.824213) (xy 3.61368 1.45937) (xy 3.978523 1.45937) (xy 4.343366 1.45937) (xy 4.343366 1.824213)
+				(xy 4.343366 2.189056) (xy 3.978523 2.189056) (xy 3.61368 2.189056) (xy 3.61368 1.824213) (xy 2.189056 1.824213)
+				(xy 2.189056 2.189056) (xy 1.824214 2.189056) (xy 1.459371 2.189056) (xy 1.459371 2.536525) (xy 1.459371 2.883994)
+				(xy 1.094528 2.883994) (xy 0.729686 2.883994) (xy 0.729686 2.171682) (xy 0.729686 1.45937) (xy 0.364843 1.45937)
+				(xy 0 1.45937) (xy 0 1.824213) (xy 0 2.189056) (xy -0.729685 2.189056) (xy -1.45937 2.189056) (xy -1.45937 1.824213)
+				(xy -1.45937 1.45937) (xy -0.729685 1.45937) (xy 0 1.45937) (xy 0 1.094528) (xy 0 0.729685) (xy -0.364842 0.729685)
+				(xy -0.729685 0.729685) (xy -0.729685 -0.364843) (xy -0.729685 -1.459371) (xy -1.094528 -1.459371)
+				(xy -1.45937 -1.459371) (xy -1.45937 -1.094528) (xy -1.45937 -0.729686) (xy -1.824213 -0.729686)
+				(xy -2.189056 -0.729686) (xy -2.189056 -0.364843) (xy -2.189056 0) (xy -1.824213 0) (xy -1.45937 0)
+				(xy -1.45937 0.364842) (xy -1.45937 0.729685) (xy -1.824213 0.729685) (xy -2.189056 0.729685) (xy -2.189056 0.364842)
+				(xy -2.189056 0) (xy -2.536525 0) (xy -2.883994 0) (xy -2.883994 0.364842) (xy -2.883994 0.729685)
+				(xy -3.248837 0.729685) (xy -3.61368 0.729685) (xy -3.61368 1.094528) (xy -3.61368 1.45937) (xy -3.248837 1.45937)
+				(xy -2.883994 1.45937) (xy -2.883994 1.824213) (xy -2.883994 2.189056) (xy -3.248837 2.189056) (xy -3.61368 2.189056)
+				(xy -3.61368 3.26621) (xy -3.61368 3.61368) (xy -2.883994 3.61368) (xy -2.883994 2.883994) (xy -2.536525 2.883994)
+				(xy -2.189056 2.883994) (xy -2.189056 3.61368) (xy -1.45937 3.61368) (xy -1.45937 2.883994) (xy -0.729685 2.883994)
+				(xy 0 2.883994) (xy 0 3.248837) (xy 0 3.26621) (xy 2.883995 3.26621) (xy 2.883995 2.189056) (xy 3.248837 2.189056)
+				(xy 3.61368 2.189056) (xy 3.61368 2.536525) (xy 3.61368 2.883994) (xy 3.978523 2.883994) (xy 4.343366 2.883994)
+				(xy 4.343366 3.248837) (xy 4.343366 3.61368) (xy 3.978523 3.61368) (xy 3.61368 3.61368) (xy 3.61368 3.978522)
+				(xy 3.61368 4.343365) (xy 3.248837 4.343365) (xy 2.883995 4.343365) (xy 2.883995 3.26621) (xy 0 3.26621)
+				(xy 0 3.61368) (xy 0.364843 3.61368) (xy 0.729686 3.61368) (xy 0.729686 3.978522) (xy 1.459371 3.978522)
+				(xy 1.459371 3.61368) (xy 1.824214 3.61368) (xy 2.189056 3.61368) (xy 2.189056 3.978522) (xy 2.189056 4.343365)
+				(xy 1.824214 4.343365) (xy 1.459371 4.343365) (xy 1.459371 3.978522) (xy 0.729686 3.978522) (xy 0.729686 4.343365)
+				(xy 0.364843 4.343365) (xy 0 4.343365) (xy 0 3.978522) (xy 0 3.61368) (xy -0.364842 3.61368) (xy -0.729685 3.61368)
+				(xy -0.729685 3.978522) (xy -0.729685 4.343365) (xy -1.094528 4.343365) (xy -1.45937 4.343365) (xy -1.45937 3.61368)
+				(xy -2.189056 3.61368) (xy -2.189056 4.343365) (xy -2.536525 4.343365) (xy -2.883994 4.343365) (xy -2.883994 3.61368)
+				(xy -3.61368 3.61368) (xy -3.61368 4.343365) (xy -3.978522 4.343365) (xy -4.343365 4.343365) (xy -4.343365 0)
+				(xy -5.003556 0) (xy -5.003556 5.003556) (xy 0 5.003556) (xy 5.003557 5.003556)
+			)
+			(stroke
+				(width 0)
+				(type solid)
+			)
+			(fill solid)
+			(layer "B.SilkS")
 		)
 	)
